File: HW/pcb/Buzzer.sch (KiCad schematic (older format))
At the start: 5 parts, among them Q3 Q_NMOS_GSD

Commit message: Committing temporary PCB changes
Parts:
- BZ1: footprint Buzzers_Beepers:MagneticBuzzer_ProSignal_ABT-410-RC -> Buzzer_Beeper:MagneticBuzzer_ProSignal_ABT-410-RC
- Q3: footprint TO_SOT_Packages_SMD:SOT-23_Handsoldering -> Package_TO_SOT_SMD:SOT-23_Handsoldering
- R19, R20, R21: footprint Resistors_SMD:R_1206_HandSoldering -> Resistor_SMD:R_1206_3216Metric_Pad1.30x1.75mm_HandSolder
Changed lines of the file:
@@
 F 0 "BZ1" H 4975 2525 50  0000 L CNN
 F 1 "Buzzer" H 4975 2425 50  0000 L CNN
-F 2 "Buzzers_Beepers:MagneticBuzzer_ProSignal_ABT-410-RC" V 4800 2575 50  0001 C CNN
+F 2 "Buzzer_Beeper:MagneticBuzzer_ProSignal_ABT-410-RC" V 4800 2575 50  0001 C CNN
 F 3 "" V 4800 2575 50  0001 C CNN
 	1    4825 2475
@@
 F 0 "Q3" H 4800 3350 50  0000 L CNN
 F 1 "Q_NMOS_GSD" H 4800 3250 50  0000 L CNN
-F 2 "TO_SOT_Packages_SMD:SOT-23_Handsoldering" H 4800 3400 50  0001 C CNN
+F 2 "Package_TO_SOT_SMD:SOT-23_Handsoldering" H 4800 3400 50  0001 C CNN
 F 3 "" H 4600 3300 50  0001 C CNN
 	1    4600 3300
@@
 F 0 "R21" V 4780 2800 50  0000 C CNN
 F 1 "12" V 4700 2800 50  0000 C CNN
-F 2 "Resistors_SMD:R_1206_HandSoldering" V 4630 2800 50  0001 C CNN
+F 2 "Resistor_SMD:R_1206_3216Metric_Pad1.30x1.75mm_HandSolder" V 4630 2800 50  0001 C CNN
 F 3 "" H 4700 2800 50  0001 C CNN
 	1    4700 2800
@@
 F 0 "R20" V 4405 3500 50  0000 C CNN
 F 1 "100k" V 4325 3500 50  0000 C CNN
-F 2 "Resistors_SMD:R_1206_HandSoldering" V 4255 3500 50  0001 C CNN
+F 2 "Resistor_SMD:R_1206_3216Metric_Pad1.30x1.75mm_HandSolder" V 4255 3500 50  0001 C CNN
 F 3 "" H 4325 3500 50  0001 C CNN
 	1    4325 3500
@@
 F 0 "R19" V 4155 3300 50  0000 C CNN
 F 1 "12" V 4075 3300 50  0000 C CNN
-F 2 "Resistors_SMD:R_1206_HandSoldering" V 4005 3300 50  0001 C CNN
+F 2 "Resistor_SMD:R_1206_3216Metric_Pad1.30x1.75mm_HandSolder" V 4005 3300 50  0001 C CNN
 F 3 "" H 4075 3300 50  0001 C CNN
 	1    4075 3300
@@
 $EndComp
 Wire Wire Line
-	4225 3300 4400 3300
+	4225 3300 4325 3300
 Wire Wire Line
 	4325 3350 4325 3300
@@
 	4325 3650 4325 3700
 Wire Wire Line
-	4325 3700 4700 3700
+	4325 3700 4500 3700
 Wire Wire Line
 	4700 3700 4700 3500
@@
 Wire Wire Line
 	4500 3875 4625 3875
+Wire Wire Line
+	4325 3300 4400 3300
+Wire Wire Line
+	4500 3700 4700 3700
 $EndSCHEMATC
