File: HW/pcb/RTD_temp_sense.sch (KiCad schematic (older format))
At the start: 7 parts, among them Q2 BC807

Commit message: Committing temporary PCB changes
Parts:
- C17: footprint Capacitors_SMD:C_1206_HandSoldering -> Capacitor_SMD:C_1206_3216Metric_Pad1.33x1.80mm_HandSolder
- Q2: footprint TO_SOT_Packages_SMD:SOT-23_Handsoldering -> Package_TO_SOT_SMD:SOT-23_Handsoldering
- R1, R17, R2: footprint Resistors_SMD:R_1206_HandSoldering -> Resistor_SMD:R_1206_3216Metric_Pad1.30x1.75mm_HandSolder
Changed lines of the file:
@@
 F 0 "R17" V 2780 2300 50  0000 C CNN
 F 1 "2k7" V 2700 2300 50  0000 C CNN
-F 2 "Resistors_SMD:R_1206_HandSoldering" V 2630 2300 50  0001 C CNN
+F 2 "Resistor_SMD:R_1206_3216Metric_Pad1.30x1.75mm_HandSolder" V 2630 2300 50  0001 C CNN
 F 3 "" H 2700 2300 50  0001 C CNN
 	1    2700 2300
@@
 F 0 "C17" H 3000 3300 50  0000 L CNN
 F 1 "10nF" H 3000 3100 50  0000 L CNN
-F 2 "Capacitors_SMD:C_1206_HandSoldering" H 3013 3050 50  0001 C CNN
+F 2 "Capacitor_SMD:C_1206_3216Metric_Pad1.33x1.80mm_HandSolder" H 3013 3050 50  0001 C CNN
 F 3 "" H 2975 3200 50  0001 C CNN
 	1    2975 3200
@@
 F 0 "Q2" H 2800 2825 50  0000 L CNN
 F 1 "BC807" H 2800 2750 50  0000 L CNN
-F 2 "TO_SOT_Packages_SMD:SOT-23_Handsoldering" H 2800 2675 50  0001 L CIN
+F 2 "Package_TO_SOT_SMD:SOT-23_Handsoldering" H 2800 2675 50  0001 L CIN
 F 3 "" H 2600 2750 50  0001 L CNN
 	1    2600 2750
@@
 F 0 "R2" V 2780 1925 50  0000 C CNN
 F 1 "200" V 2700 1925 50  0000 C CNN
-F 2 "Resistors_SMD:R_1206_HandSoldering" V 2630 1925 50  0001 C CNN
+F 2 "Resistor_SMD:R_1206_3216Metric_Pad1.30x1.75mm_HandSolder" V 2630 1925 50  0001 C CNN
 F 3 "" H 2700 1925 50  0001 C CNN
 	1    2700 1925
@@
 F 0 "R1" V 2180 3050 50  0000 C CNN
 F 1 "270" V 2100 3050 50  0000 C CNN
-F 2 "Resistors_SMD:R_1206_HandSoldering" V 2030 3050 50  0001 C CNN
+F 2 "Resistor_SMD:R_1206_3216Metric_Pad1.30x1.75mm_HandSolder" V 2030 3050 50  0001 C CNN
 F 3 "" H 2100 3050 50  0001 C CNN
 	1    2100 3050
