File: HW/pcb/panel.kicad_pcb (KiCad board)
At the start: 2 copper layers, 117.6 x 112.5 mm, 90 parts, among them J1 Conn_01x02_Male, J14 TEST_1P, J15 Conn_01x07_Female, J16 Conn_01x16, J17 TEST_1P, J19 Conn_01x01, J2 USART test points, J23 Conn_01x01, J24 Conn_01x01, J25 Conn_01x01, J26 Conn_01x01, J27 Conn_01x01, J28 Conn_01x01, J29 Conn_01x01, J3 Conn_01x02_Male, J30 Conn_01x01, J31 Conn_01x01, J4 Conn_01x08_Female, J5 Conn_02x03_Odd_Even, J6 Conn_01x02_Male, J7 Conn_01x03_Male, J8 Conn_01x03_Male, J9 Jack-DC, Q1 Q_NMOS_GSD, Q2 BC807, Q3 Q_NMOS_GSD, Q4 Q_NMOS_GSD, SW1 SW_Push_Dual_OWN, SW2 SW_Push_Dual_OWN, SW3 SW_Push_Dual_OWN, SW4 Rotary_Encoder_With_CaseHolder, U3 ATMEGA128-16AU, Y1 Crystal_GND24_Small

Commit message: Committing temporary PCB changes
Parts:
- removed D4, D5, D6, D7: blue, LEDs:LED_1206_HandSoldering
- removed D9: 5VBreakdown_Zener, Diodes_SMD:D_MiniMELF_Handsoldering
- added J10: current sense, Connector_PinHeader_2.54mm:PinHeader_1x02_P2.54mm_Vertical, F.Cu at (197.0, 68.7)
- added J11: GND conn, Connector_PinHeader_2.54mm:PinHeader_1x04_P2.54mm_Vertical, F.Cu at (88.4, 122.6)
- added LED1: blue, LED_SMD:LED_1206_3216Metric_Castellated, F.Cu at (182.3, 99.4)
- added LED2: blue, LED_SMD:LED_1206_3216Metric_Castellated, F.Cu at (177.3, 99.4)
- added LED3: blue, LED_SMD:LED_1206_3216Metric_Castellated, F.Cu at (172.3, 99.4)
- added LED4: blue, LED_SMD:LED_1206_3216Metric_Castellated, F.Cu at (167.3, 99.4)
- 18pF1, 18pF2: footprint Capacitors_SMD:C_1206_HandSoldering -> Capacitor_SMD:C_0805_2012Metric_Pad1.18x1.45mm_HandSolder
- BZ1: footprint Buzzers_Beepers:MagneticBuzzer_ProSignal_ABT-410-RC -> Buzzer_Beeper:MagneticBuzzer_ProSignal_ABT-410-RC
- C10, C11, C12, C13, C14, C15, C16, C17, C3, C5, C8, C9: footprint Capacitors_SMD:C_1206_HandSoldering -> Capacitor_SMD:C_1206_3216Metric_Pad1.33x1.80mm_HandSolder
- C2: footprint Capacitors_SMD:C_1206_HandSoldering -> Capacitor_SMD:C_1206_3216Metric_Pad1.33x1.80mm_HandSolder; moved to F.Cu
- D8: footprint Diodes_SMD:D_MiniMELF_Handsoldering -> Diode_SMD:D_MiniMELF_Handsoldering
- J1, J6: footprint Pin_Headers:Pin_Header_Straight_1x02_Pitch2.54mm -> Connector_PinHeader_2.54mm:PinHeader_1x02_P2.54mm_Vertical
- J15: footprint Socket_Strips:Socket_Strip_Straight_1x07_Pitch2.54mm -> Connector_PinSocket_2.54mm:PinSocket_1x07_P2.54mm_Vertical
- J16: footprint Socket_Strips:Socket_Strip_Straight_1x16_Pitch2.54mm -> Connector_PinSocket_2.54mm:PinSocket_1x16_P2.54mm_Vertical
- J19, J23, J28, J29, J30, J31: footprint Mounting_Holes:MountingHole_2.5mm -> MountingHole:MountingHole_2.5mm_Pad
- J2, J7, J8: footprint Pin_Headers:Pin_Header_Straight_1x03_Pitch2.54mm -> Connector_PinHeader_2.54mm:PinHeader_1x03_P2.54mm_Vertical
- J24, J25, J26, J27: footprint Mounting_Holes:MountingHole_3.5mm -> MountingHole:MountingHole_3.5mm_Pad
- J4: value Conn_01x08_Female -> uart_conn; footprint Socket_Strips:Socket_Strip_Straight_1x08_Pitch2.54mm -> Connector_PinSocket_2.54mm:PinSocket_1x06_P2.54mm_Vertical
- J5: footprint Pin_Headers:Pin_Header_Straight_2x03_Pitch2.54mm -> Connector_PinHeader_2.54mm:PinHeader_2x03_P2.54mm_Vertical
- J9: value Jack-DC -> USB_B_Mini; footprint Connectors:JACK_ALIM -> Connector_USB:USB_Mini-B_Lumberg_2486_01_Horizontal
- Q1, Q2, Q3, Q4: footprint TO_SOT_Packages_SMD:SOT-23_Handsoldering -> Package_TO_SOT_SMD:SOT-23_Handsoldering
- R1, R10, R13, R14, R15, R16, R17, R19, R2, R20, R21, R22, R23, R24, R25, R26, R27, R28, R29, R30, R5, R6, R7, R8, R9: footprint Resistors_SMD:R_1206_HandSoldering -> Resistor_SMD:R_1206_3216Metric_Pad1.30x1.75mm_HandSolder
- RV1, RV2, RV4: footprint Potentiometers:Potentiometer_Trimmer_ACP_CA9v_Horizontal_Px10.0mm_Py5.0mm -> Potentiometer_THT:Potentiometer_ACP_CA9-V10_Vertical
- SW1, SW2: footprint Buttons_Switches_THT:SW_TH_Tactile_Omron_B3F-10xx -> Button_Switch_THT:SW_TH_Tactile_Omron_B3F-10xx
- U3: footprint Housings_QFP:TQFP-64_14x14mm_Pitch0.8mm -> Package_QFP:TQFP-64_14x14mm_P0.8mm
- Y1: footprint Crystals:Crystal_SMD_3225-4pin_3.2x2.5mm -> Crystal:Crystal_SMD_3225-4Pin_3.2x2.5mm
- moved D8 11.4 mm to (183.1, 55.2), turned to 90 degrees
- moved R7 11.1 mm to (182.3, 99.5)
- moved J9 9.94 mm to (194.7, 54.9), turned to 90 degrees
- moved R6 8.79 mm to (177.3, 99.5)
- moved R8 6.44 mm to (172.3, 99.5)
- moved J4 5.08 mm to (86.1, 65.4)
- moved R9 3.77 mm to (167.3, 99.4)
- moved J14 3.01 mm to (185.6, 133.8)
- moved 18pF1 2.28 mm to (128.9, 108.3), turned to 270 degrees
- moved C2 2.22 mm to (96.5, 120.3)
- moved J1 2.13 mm to (109.1, 104.1)
- moved 18pF2 2.12 mm to (132.5, 108.3), turned to 270 degrees
- moved F1 1.78 mm to (94.8, 116.2)
- moved J25 1.67 mm to (193.8, 141.7)
- moved J27 1.64 mm to (88.7, 141.7)
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Connections:
- D8 pad 2: Net-(D8-Pad2) -> /Input_filter/DC_2
- J4 pad 2: Net-(J4-Pad2) -> Net-(J4-Pad1)
- J4 pad 4: Net-(J4-Pad3) -> Net-(J2-Pad2)
- J4 pad 5: Net-(J4-Pad5) -> MISO
- J4 pad 6: Net-(J2-Pad2) -> GNDREF
- J9 pad 2: /Input_filter/DC_2 -> Net-(J9-Pad2)
- J9 pad 3: /Input_filter/DC_2 -> Net-(J9-Pad3)
- L2 pad 1: /Input_filter/DC_1 -> Net-(J10-Pad1)
Routing:
- net GNDREF: track 256.1 -> 100.6 mm, vias 39 -> 131
- net /Input_filter/DC_2: track 37.0 -> 61.6 mm
- net Net-(J10-Pad1): track 0.00 -> 22.3 mm
- net /Input_filter/DC_1: track 8.87 -> 19.2 mm
- net LED1: track 65.2 -> 58.4 mm
- net Net-(Q3-Pad3): track 10.3 -> 3.84 mm
- net Net-(Q3-Pad1): track 8.82 -> 14.2 mm
- net Net-(D8-Pad2): track 4.37 -> 0.00 mm
- net LED2: track 55.6 -> 51.9 mm
- net LED3: track 47.5 -> 43.9 mm
- net Capacitive_button_1: track 57.8 -> 54.7 mm
- net Net-(J4-Pad3): track 2.54 -> 0.00 mm
- net Net-(J4-Pad1): track 0.00 -> 2.54 mm
- net Net-(C13-Pad1): track 12.8 -> 10.7 mm
- net MISO: track 108.0 -> 110.1 mm
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