File: HW/pcb/panel.sch (KiCad schematic (older format))
At the start: 54 parts, among them J1 Conn_01x02_Male, J14 TEST_1P, J17 TEST_1P, J2 USART test points, J24 Conn_01x01, J25 Conn_01x01, J26 Conn_01x01, J27 Conn_01x01, J3 Conn_01x02_Male, J4 Conn_01x08_Female, J5 Conn_02x03_Odd_Even, J6 Conn_01x02_Male, J7 Conn_01x03_Male, J8 Conn_01x03_Male, J9 Jack-DC, SW1 SW_Push_Dual_OWN, SW2 SW_Push_Dual_OWN, SW3 SW_Push_Dual_OWN, SW4 Rotary_Encoder_With_CaseHolder, U3 ATMEGA128-16AU, Y1 Crystal_GND24_Small

Commit message: Committing temporary PCB changes
Parts:
- removed J4: Conn_01x08_Female, Socket_Strips:Socket_Strip_Straight_1x08_Pitch2.54mm, symbol panel-rescue:Conn_01x08_Female
- removed J9: Jack-DC, Connectors:JACK_ALIM, symbol panel-rescue:Jack-DC
- added J11: GND conn, Connector_PinHeader_2.54mm:PinHeader_1x04_P2.54mm_Vertical, symbol Connector:Conn_01x04_Male
- added J4: uart_conn, Connector_PinSocket_2.54mm:PinSocket_1x06_P2.54mm_Vertical, symbol Connector:Conn_01x06_Female
- added J9: USB_B_Mini, Connector_USB:USB_Mini-B_Lumberg_2486_01_Horizontal, symbol Connector:USB_B_Mini
- 18pF1, 18pF2: footprint Capacitors_SMD:C_1206_HandSoldering -> Capacitor_SMD:C_0805_2012Metric_Pad1.18x1.45mm_HandSolder
- C10, C11, C12, C13, C2, C3, C5, C8, C9: footprint Capacitors_SMD:C_1206_HandSoldering -> Capacitor_SMD:C_1206_3216Metric_Pad1.33x1.80mm_HandSolder
- J1, J6: footprint Pin_Headers:Pin_Header_Straight_1x02_Pitch2.54mm -> Connector_PinHeader_2.54mm:PinHeader_1x02_P2.54mm_Vertical
- J2, J7, J8: footprint Pin_Headers:Pin_Header_Straight_1x03_Pitch2.54mm -> Connector_PinHeader_2.54mm:PinHeader_1x03_P2.54mm_Vertical
- J24, J25, J26, J27: footprint Mounting_Holes:MountingHole_3.5mm -> MountingHole:MountingHole_3.5mm_Pad
- J5: footprint Pin_Headers:Pin_Header_Straight_2x03_Pitch2.54mm -> Connector_PinHeader_2.54mm:PinHeader_2x03_P2.54mm_Vertical
- LED1: renamed from D4; footprint LEDs:LED_1206_HandSoldering -> LED_SMD:LED_1206_3216Metric_Castellated
- LED2: renamed from D5; footprint LEDs:LED_1206_HandSoldering -> LED_SMD:LED_1206_3216Metric_Castellated
- LED3: renamed from D6; footprint LEDs:LED_1206_HandSoldering -> LED_SMD:LED_1206_3216Metric_Castellated
- LED4: renamed from D7; footprint LEDs:LED_1206_HandSoldering -> LED_SMD:LED_1206_3216Metric_Castellated
- R10, R13, R14, R15, R16, R22, R23, R30, R5, R6, R7, R8, R9: footprint Resistors_SMD:R_1206_HandSoldering -> Resistor_SMD:R_1206_3216Metric_Pad1.30x1.75mm_HandSolder
- RV1, RV2: footprint Potentiometers:Potentiometer_Trimmer_ACP_CA9v_Horizontal_Px10.0mm_Py5.0mm -> Potentiometer_THT:Potentiometer_ACP_CA9-V10_Vertical
- SW1, SW2: footprint Buttons_Switches_THT:SW_TH_Tactile_Omron_B3F-10xx -> Button_Switch_THT:SW_TH_Tactile_Omron_B3F-10xx
- U3: footprint Housings_QFP:TQFP-64_14x14mm_Pitch0.8mm -> Package_QFP:TQFP-64_14x14mm_P0.8mm
- Y1: footprint Crystals:Crystal_SMD_3225-4pin_3.2x2.5mm -> Crystal:Crystal_SMD_3225-4Pin_3.2x2.5mm
Connections:
- net GNDREF: now also J11.1 (Pin_1), J11.2 (Pin_2), J11.3 (Pin_3), J11.4 (Pin_4), J4.6 (Pin_6)
- net Input_filter/DC_1: now also J9.1 (VBUS)
- net Input_filter/DC_2: now also J9.5 (GND), J9.6 (Shield)
- net MISO: now also J4.5 (Pin_5)
- net at J2.2 (Pin_2), R5.2: now also J4.4 (Pin_4)
- new net: J4.1 (Pin_1), J4.2 (Pin_2)
- no-connect marks 33 -> 34
